Commit message: Fixed panda-robotiq urdf

File: mani_skill/assets/robots/panda/panda_robotiq_85_alt_2.urdf (robot description, URDF)
Before this commit: robot panda, 21 links, 20 joints
Links:
- removed link robotiq_hand_tcp
Joints:
- removed joint robotiq_hand_tcp_joint
- joint panda_joint_ee: origin xyz=0 0 0.045 rpy=0 0 0 -> xyz=0 0 0.10 rpy=0 0 0

Commit message: Added gripper tcp link

File: mani_skill/assets/robots/panda/panda_robotiq_85_alt_2.urdf (robot description, URDF)
Before this commit: robot panda, 20 links, 19 joints
Links:
- added link robotiq_hand_tcp
Joints:
- added joint robotiq_hand_tcp_joint: type fixed, parent robotiq_arg2f_base_link, child robotiq_hand_tcp, origin xyz=0 0 0.174 rpy=0 0 0
