Commit message: Match urdf file to DROID demo repo: https://github.com/rerun-io/python-example-droid-dataset/tree/master

File: mani_skill/assets/robots/panda/panda_robotiq_85.urdf (robot description, URDF)
Before this commit: robot panda, 21 links, 20 joints
Joints:
- joint panda_joint_ee: origin xyz=0 0 0.10 rpy=0 0 0 -> xyz=0 0 0.107 rpy=0 0 0

Commit message: Create motion planning scripts for pick carrot task

File: mani_skill/assets/robots/panda/panda_robotiq_85.urdf (robot description, URDF)
Before this commit: robot panda, 21 links, 20 joints
Links:
- link left_inner_finger: geometry collision mesh filename=robotiq-2f/meshes/collision/robotiq_arg2f_85_inner_finger.s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 scale=0.001 0.001 0.001; visual mesh filename=robotiq-2f/meshes/visual/robotiq_arg2f_85_inner_finger.dae scale=0.001 0.001 0.001
- link left_outer_finger: geometry collision mesh filename=robotiq-2f/meshes/collision/robotiq_arg2f_85_outer_finger.s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 scale=0.001 0.001 0.001; visual mesh filename=robotiq-2f/meshes/visual/robotiq_arg2f_85_outer_finger.dae scale=0.001 0.001 0.001
- link right_inner_finger: geometry collision mesh filename=robotiq-2f/meshes/collision/robotiq_arg2f_85_inner_finger.s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 scale=0.001 0.001 0.001; visual mesh filename=robotiq-2f/meshes/visual/robotiq_arg2f_85_inner_finger.dae scale=0.001 0.001 0.001
- link right_outer_finger: geometry collision mesh filename=robotiq-2f/meshes/collision/robotiq_arg2f_85_outer_finger.s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 scale=0.001 0.001 0.001; visual mesh filename=robotiq-2f/meshes/visual/robotiq_arg2f_85_outer_finger.dae scale=0.001 0.001 0.001
Joints:
- joint robotiq_hand_tcp_joint: origin xyz=0 0 0.174 rpy=0 0 0 -> xyz=0 0 0.15 rpy=0 0 0

Commit message: Testing out maniskill to openx data conversion

File: mani_skill/assets/robots/panda/panda_robotiq_85.urdf (robot description, URDF)
Before this commit: robot panda, 21 links, 20 joints
Links:
- link panda_link_ee: mass 0 -> None
